File: Baseboards/SoMProgrammerNTester/SoMProgrammerNTester.kicad_sch (KiCad schematic)
At the start: 34 parts, among them J1 SoM Connector, J2 Conn_01x12_Pin, SW1 CAS-D20TB, SW2 CAS-D20TB, U1 SN74LVC00APWE4, U2 74AUP1G04

Commit message: Created Version with 0402 components
Parts:
- J1: Mouser Part Number 571-1-1473005-1 -> 571-1473005-1
Changed lines of the file:
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@@
 			)
 		)
-		(property "Mouser Part Number" "571-1-1473005-1"
+		(property "Mouser Part Number" "571-1473005-1"
 			(at 69.85 82.55 0)
 			(effects
@@
 			)
 		)
-		(property "Mouser Part Number" "571-1-1473005-1"
+		(property "Mouser Part Number" "571-1473005-1"
 			(at 156.21 48.26 0)
 			(effects
