File: Baseboards/SoMProgrammerNTester/Southbank.kicad_sch (KiCad schematic)
At the start: 36 parts, among them J1 SoM Connector

Commit message: Created Version with 0402 components
Parts:
- J1: Mouser Part Number 571-1-1473005-1 -> 571-1473005-1
Changed lines of the file:
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@@
 			)
 		)
-		(property "Mouser Part Number" "571-1-1473005-1"
+		(property "Mouser Part Number" "571-1473005-1"
 			(at 135.89 73.66 0)
 			(effects
