File: SoM/FPGA_IO_Config.kicad_sch (KiCad schematic)
At the start: 1 part, among them U1 CCGM1A1

Commit message: Created Version with 0402 components
Parts:
- U1: Mouser Part Number (none) -> CCGM1A1-BGA324; Part Number (none) -> CCGM1A1-BGA324
