File: SoM/SODIM.kicad_sch (KiCad schematic)
At the start: 2 parts, among them J1 SODIMM-200_Split

Commit message: Created Version with 0402 components
Parts:
- R25: footprint Resistor_SMD:R_0201_0603Metric -> Resistor_SMD:R_0402_1005Metric; Mouser Part Number 71-CRCW0201100RFNED -> MCS04020C1000FE000; Part Number (none) -> MCS04020C1000FE000
